File: pulse-delay.kicad_pcb (KiCad board)
At the start: 2 copper layers, 11 parts, among them J1 Conn_02x05_Odd_Even

Commit message: pcb ready for v0
Parts:
- added C3: 10n, Capacitor_SMD:C_0805_2012Metric, F.Cu at (117.4, 110.4)
- added C4: 100n, Capacitor_SMD:C_0805_2012Metric, F.Cu at (125.0, 121.3)
- added C5: 1u box, Capacitor_THT:C_Rect_L7.2mm_W5.5mm_P5.00mm_FKS2_FKP2_MKS2_MKP2, B.Cu at (118.6, 122.0)
- added C6: 1u box, Capacitor_THT:C_Rect_L7.2mm_W5.5mm_P5.00mm_FKS2_FKP2_MKS2_MKP2, B.Cu at (129.0, 114.5)
- added C7: 100n, Capacitor_SMD:C_0805_2012Metric, F.Cu at (121.7, 111.2)
- added D3: 1N4148, Diode_SMD:D_SOD-323_HandSoldering, F.Cu at (117.1, 112.9)
- added D4: 1N4148, Diode_SMD:D_SOD-323_HandSoldering, F.Cu at (122.7, 106.6)
- added D5: LED, LED_THT:LED_D3.0mm, F.Cu at (110.5, 121.5)
- added H10: out, Eurorack:Mech-AudioJack-Hole-Output-Gate, F.Cu at (101.1, 152.3)
- added H11: delay, Eurorack:Mech-Potentiometer-Hole_level_90deg, F.Cu at (125.4, 144.2)
- added H12: width, Eurorack:Mech-Potentiometer-Hole_level_90deg, F.Cu at (151.2, 144.2)
- added H13: led, Eurorack:Mech-LED-Hole-3mm-Bezel, F.Cu at (111.8, 155.2)
- added H9: in, Eurorack:Mech-AudioJack-Hole-Input-Gate, F.Cu at (101.1, 141.1)
- added J2: AudioJack2_SwitchT, Eurorack:AudioJack2_Tayda_A-2566, F.Cu at (101.1, 107.3)
- added J3: AudioJack2_SwitchT, Eurorack:AudioJack2_Tayda_A-2566, F.Cu at (101.1, 118.5)
- added Q1: BCM847, Package_SO:TSOP-6_1.65x3.05mm_P0.95mm, F.Cu at (125.1, 111.2)
- added R10: 10K, Resistor_SMD:R_0805_2012Metric, F.Cu at (107.7, 122.1)
- added R3: 100K, Resistor_SMD:R_0805_2012Metric, F.Cu at (116.6, 106.3)
- added R4: 22K, Resistor_SMD:R_0805_2012Metric, F.Cu at (119.1, 106.3)
- added R5: 22K, Resistor_SMD:R_0805_2012Metric, F.Cu at (128.5, 111.2)
- added R6: 10K, Resistor_SMD:R_0805_2012Metric, F.Cu at (112.8, 106.6)
- added R7: 10K, Resistor_SMD:R_0805_2012Metric, F.Cu at (132.4, 106.3)
- added R8: 1K, Resistor_SMD:R_0805_2012Metric, F.Cu at (115.8, 121.6)
- added R9: 1.8K, Resistor_SMD:R_0805_2012Metric, F.Cu at (110.5, 118.3)
- added RV1: A1M, Eurorack:Potentiometer_RV16AF-41-15R1, F.Cu at (125.4, 110.5)
- added RV2: A1M, Eurorack:Potentiometer_RV16AF-41-15R1, F.Cu at (151.2, 110.5)
- added U1: 4538, Package_SO:TSSOP-16_4.4x5mm_P0.65mm, F.Cu at (124.0, 117.1)
- moved H3 181.3 mm to (154.8, 163.8)
- moved H2 160.2 mm to (154.8, 130.0)
- moved H4 146.9 mm to (99.0, 163.7)
- moved H1 129.0 mm to (99.1, 130.1)
- moved J1 114.0 mm to (146.1, 118.0), turned to 0 degrees
- moved D1 106.7 mm to (141.7, 117.5), turned to -90 degrees
- moved C1 105.6 mm to (138.3, 120.6), turned to 0 degrees
- moved R2 104.1 mm to (142.8, 114.2), turned to 0 degrees
- moved R1 101.2 mm to (142.8, 111.7), turned to 0 degrees
- moved D2 95.9 mm to (141.7, 108.4), turned to -90 degrees
- moved C2 90.7 mm to (140.7, 105.1), turned to 180 degrees
Routing:
- net +12V: track 14.2 -> 95.1 mm, vias 0 -> 1
- net GND: track 41.0 -> 98.7 mm, vias 0 -> 3
- net Net-(Q1B-B2): track 0.00 -> 28.5 mm
- net Net-(U1B-RxCx): track 0.00 -> 19.0 mm
- net Net-(Q1B-E2): track 0.00 -> 16.3 mm, vias 0 -> 2
- net Net-(U1A-RxCx): track 0.00 -> 15.1 mm
- net Net-(D3-A): track 0.00 -> 15.1 mm
- net Net-(Q1A-C1): track 0.00 -> 12.4 mm
- net Net-(D4-K): track 0.00 -> 12.0 mm
- net Net-(J3-PadT): track 0.00 -> 11.2 mm
- net Net-(U1A-Clk+): track 0.00 -> 8.77 mm
- net Net-(D3-K): track 0.00 -> 6.31 mm
- net Net-(R6-Pad2): track 0.00 -> 3.23 mm
- net Net-(D5-A): track 0.00 -> 3.19 mm
- net Net-(R7-Pad2): track 0.00 -> 2.69 mm
- added copper zone on B.Cu, net /FACE
- added copper zone on F.Cu, net /FACE
- added copper zone on B.Cu, net GND
- added copper zone on F.Cu, net GND
Other:
- board outline added: 65.7 x 64.7 mm
- board text added: "pulse delay"
- board text added: "thismatters/pulse-delay/v0"

Commit message: update bom
Parts:
- D5: value LED -> LED_GREEN
Changed lines of the file:
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@@
     (descr "TSSOP, 16 Pin (JEDEC MO-153 Var AB https://www.jedec.org/document_search?search_api_views_fulltext=MO-153), generated with kicad-footprint-generator ipc_gullwing_generator.py")
     (tags "TSSOP SO")
-    (property "Sheetfile" "pulse-delay.kicad_sch")
-    (property "Sheetname" "")
+    (property "PartNum" "595-CD14538BPWR")
+    (property "Sheetfile" "pulse-delay.kicad_sch")
+    (property "Sheetname" "")
+    (property "Vendor" "Mouser")
     (property "ki_description" "Monostable")
     (property "ki_keywords" "CMOS")
@@
     (descr "TSOP-6 package (comparable to TSOT-23), https://www.vishay.com/docs/71200/71200.pdf")
     (tags "Jedec MO-193C TSOP-6L")
-    (property "Sheetfile" "pulse-delay.kicad_sch")
-    (property "Sheetname" "")
+    (property "PartNum" "771-BCM847DS135")
+    (property "Sheetfile" "pulse-delay.kicad_sch")
+    (property "Sheetname" "")
+    (property "Vendor" "Mouser")
     (property "ki_description" "Dual NPN transistor, 6 pin package")
     (property "ki_keywords" "transistor NPN")
@@
         (effects (font (size 1 1) (thickness 0.15)))
     )
-    (fp_text value "LED" (at 1.27 2.96) (layer "F.Fab")
-        (effects (font (size 1 1) (thickness 0.15)))
-    )
+    (fp_text value "LED_GREEN" (at 1.27 2.96) (layer "F.Fab")
+        (effects (font (size 1 1) (thickness 0.15)))
+    )
