File: pulse-delay.kicad_sch (KiCad schematic)
At the start: 48 parts, among them J1 Conn_02x05_Odd_Even, J2 AudioJack2_SwitchT, J3 AudioJack2_SwitchT, M1 Standoff, M2 Standoff, M3 Screw, M4 Screw, M5 Screw, M6 Screw, Q1 BCM847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

Commit message: pcb ready for v0
Parts:
- removed H5, H6, H7, H8: Standoff, MountingHole:MountingHole_2.7mm_M2.5, symbol Mechanical:MountingHole
- removed M1, M2: Standoff, Eurorack:Standoff_M2.5x0.45-11mm, symbol Eurorack:Standoff
- removed M3, M4, M5, M6: Screw, Eurorack:Screw_M2.5x0.45-6mm, symbol Eurorack:Screw
- C3, C4, C7: footprint (none) -> Capacitor_SMD:C_0805_2012Metric
- C5, C6: footprint (none) -> Capacitor_THT:C_Rect_L7.2mm_W5.5mm_P5.00mm_FKS2_FKP2_MKS2_MKP2
- D3, D4: footprint (none) -> Diode_SMD:D_SOD-323_HandSoldering
- D5: footprint (none) -> LED_THT:LED_D3.0mm
- J2, J3: footprint (none) -> Eurorack:AudioJack2_Tayda_A-2566
- Q1: footprint (none) -> Package_SO:TSOP-6_1.65x3.05mm_P0.95mm
- R10, R3, R4, R5, R6, R7, R8, R9: footprint (none) -> Resistor_SMD:R_0805_2012Metric
- RV1, RV2: footprint (none) -> Eurorack:Potentiometer_RV16AF-41-15R1
- U1: footprint (none) -> Package_SO:TSSOP-16_4.4x5mm_P0.65mm
Connections:
- net +12V: now also RV1.3, RV2.3; no longer RV1.1, RV2.1
- net at R7.2: now also RV2.1; no longer RV2.3
- net at R6.2: now also RV1.1; no longer RV1.3
Other:
- note removed: "Mechanical attachment for 3 layer module"
- moved on the sheet: RV1, RV2

Commit message: update bom
Parts:
- D5: value LED -> LED_GREEN
- Q1: PartNum (none) -> 771-BCM847DS135; Vendor (none) -> Mouser
- U1: PartNum (none) -> 595-CD14538BPWR; Vendor (none) -> Mouser
Changed lines of the file:
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@@
+      (effects (font (size 1.27 1.27)) hide)
+    )
+    (property "Vendor" "Mouser" (at 220.98 38.1 0)
+      (effects (font (size 1.27 1.27)) hide)
+    )
+    (property "PartNum" "771-BCM847DS135" (at 220.98 38.1 0)
       (effects (font (size 1.27 1.27)) hide)
     )
@@
     )
     (property "Datasheet" "https://assets.nexperia.com/documents/data-sheet/HEF4538B.pdf" (at 272.415 144.78 0)
+      (effects (font (size 1.27 1.27)) hide)
+    )
+    (property "Vendor" "Mouser" (at 272.415 146.05 0)
+      (effects (font (size 1.27 1.27)) hide)
+    )
+    (property "PartNum" "595-CD14538BPWR" (at 272.415 146.05 0)
       (effects (font (size 1.27 1.27)) hide)
     )
@@
       (effects (font (size 1.27 1.27)) hide)
     )
+    (property "Vendor" "Mouser" (at 186.055 67.31 0)
+      (effects (font (size 1.27 1.27)) hide)
+    )
+    (property "PartNum" "595-CD14538BPWR" (at 186.055 67.31 0)
+      (effects (font (size 1.27 1.27)) hide)
+    )
     (pin "9")
     (pin "11")
@@
       (effects (font (size 1.27 1.27)) hide)
     )
+    (property "Vendor" "Mouser" (at 93.345 45.085 0)
+      (effects (font (size 1.27 1.27)) hide)
+    )
+    (property "PartNum" "771-BCM847DS135" (at 93.345 45.085 0)
+      (effects (font (size 1.27 1.27)) hide)
+    )
     (pin "2")
     (pin "5")
@@
       (effects (font (size 1.27 1.27)) hide)
     )
+    (property "Vendor" "Mouser" (at 136.525 67.31 0)
+      (effects (font (size 1.27 1.27)) hide)
+    )
+    (property "PartNum" "595-CD14538BPWR" (at 136.525 67.31 0)
+      (effects (font (size 1.27 1.27)) hide)
+    )
     (pin "9")
     (pin "11")
@@
       (effects (font (size 1.27 1.27)) (justify right))
     )
-    (property "Value" "LED" (at 227.33 57.4675 90)
+    (property "Value" "LED_GREEN" (at 227.33 57.4675 90)
       (effects (font (size 1.27 1.27)) (justify right))
     )
